Commit message: human

File: launch/human.right_leg.xacro (robot description, xacro)
@@ -3,5 +3,5 @@
     xmlns:xacro="http://www.ros.org/wiki/xacro">
     <!-- right leg -->
-    <xacro:macro name="uthai_right_leg" params="parent dxl_effort dxl_speed">
+    <xacro:macro name="human_right_leg" params="parent dxl_effort dxl_speed">
         <!-- right hip yaw joint -->
         <joint name="r_hip_yaw_joint" type="revolute">

File: launch/human.visuals.xacro (robot description, xacro)
@@ -6,5 +6,5 @@
         <origin xyz="0 0 0" rpy="0 0 0" />
         <geometry>
-            <mesh filename="package://meshes/base.STL" scale="1 1 1" />
+            <mesh filename="package://human/meshes/base.STL" scale="1 1 1" />
         </geometry>
         <material name="grey"/>
@@ -14,5 +14,5 @@
         <origin xyz="0 0 0" rpy="0 0 0" />
         <geometry>
-            <mesh filename="package://meshes/r_hip_yaw.STL" scale="1 1 1" />
+            <mesh filename="package://human/meshes/r_hip_yaw.STL" scale="1 1 1" />
         </geometry>
         <material name="grey"/>
@@ -22,5 +22,5 @@
         <origin xyz="0 0 0" rpy="0 0 0" />
         <geometry>
-            <mesh filename="package://meshes/r_hip_roll.STL" scale="1 1 1" />
+            <mesh filename="package://human/meshes/r_hip_roll.STL" scale="1 1 1" />
         </geometry>
         <material name="grey"/>
@@ -30,5 +30,5 @@
         <origin xyz="0 0 0" rpy="0 0 0" />
         <geometry>
-            <mesh filename="package://meshes/r_hip_pitch.STL" scale="1 1 1" />
+            <mesh filename="package://human/meshes/r_hip_pitch.STL" scale="1 1 1" />
         </geometry>
         <material name="grey"/>
@@ -38,5 +38,5 @@
         <origin xyz="0 0 0" rpy="0 0 0" />
         <geometry>
-            <mesh filename="package://meshes/r_knee_pitch.STL" scale="1 1 1" />
+            <mesh filename="package://human/meshes/r_knee_pitch.STL" scale="1 1 1" />
         </geometry>
         <material name="grey"/>
@@ -46,5 +46,5 @@
         <origin xyz="0 0 0" rpy="0 0 0" />
         <geometry>
-            <mesh filename="package://meshes/r_ankle_pitch.STL" scale="1 1 1" />
+            <mesh filename="package://human/meshes/r_ankle_pitch.STL" scale="1 1 1" />
         </geometry>
         <material name="grey"/>
@@ -54,5 +54,5 @@
         <origin xyz="0 0 0" rpy="0 0 0" />
         <geometry>
-            <mesh filename="package://meshes/r_ankle_roll.STL" scale="1 1 1" />
+            <mesh filename="package://human/meshes/r_ankle_roll.STL" scale="1 1 1" />
         </geometry>
         <material name="grey"/>
@@ -62,5 +62,5 @@
         <origin xyz="0 0 0" rpy="0 0 0" />
         <geometry>
-            <mesh filename="package://meshes/l_hip_yaw.STL" scale="1 1 1" />
+            <mesh filename="package://human/meshes/l_hip_yaw.STL" scale="1 1 1" />
         </geometry>
         <material name="grey"/>
@@ -70,5 +70,5 @@
         <origin xyz="0 0 0" rpy="0 0 0" />
         <geometry>
-            <mesh filename="package://meshes/l_hip_roll.STL" scale="1 1 1" />
+            <mesh filename="package://human/meshes/l_hip_roll.STL" scale="1 1 1" />
         </geometry>
         <material name="grey"/>
@@ -78,5 +78,5 @@
         <origin xyz="0 0 0" rpy="0 0 0" />
         <geometry>
-            <mesh filename="package://meshes/l_hip_pitch.STL" scale="1 1 1" />
+            <mesh filename="package://human/meshes/l_hip_pitch.STL" scale="1 1 1" />
         </geometry>
         <material name="grey"/>
@@ -86,5 +86,5 @@
         <origin xyz="0 0 0" rpy="0 0 0" />
         <geometry>
-            <mesh filename="package://meshes/l_knee_pitch.STL" scale="1 1 1" />
+            <mesh filename="package://human/meshes/l_knee_pitch.STL" scale="1 1 1" />
         </geometry>
         <material name="grey"/>
@@ -94,5 +94,5 @@
         <origin xyz="0 0 0" rpy="0 0 0" />
         <geometry>
-            <mesh filename="package://meshes/l_ankle_pitch.STL" scale="1 1 1" />
+            <mesh filename="package://human/meshes/l_ankle_pitch.STL" scale="1 1 1" />
         </geometry>
         <material name="grey"/>
@@ -102,5 +102,5 @@
         <origin xyz="0 0 0" rpy="0 0 0" />
         <geometry>
-            <mesh filename="package://meshes/l_ankle_roll.STL" scale="1 1 1" />
+            <mesh filename="package://human/meshes/l_ankle_roll.STL" scale="1 1 1" />
         </geometry>
         <material name="grey"/>

File: launch/human.xacro (robot description, xacro)
@@ -5,5 +5,5 @@
     <!-- Import xacro file -->
     <xacro:include filename="human.materials.xacro" />
-    <!-- <xacro:include filename="human.visuals.xacro" /> -->
+    <xacro:include filename="human.visuals.xacro" />
     <xacro:include filename="human.inertia.xacro" />
     <xacro:include filename="human.transmissions.xacro" />
@@ -12,10 +12,10 @@
     <xacro:include filename="human.gazebo.xacro" />
     <!-- Used for fixing robot -->
-    <!--<link name="world"></link>
+    <link name="world"></link>
     <joint name="world_fixed" type="fixed">
         <origin xyz="0 0 0.764" rpy="0 0 0"/>
         <parent link="world"/>
         <child link="base_link"/>
-    </joint> -->
+    </joint>
     <link name="base_link"></link>
     <joint name="base_fixed" type="fixed">
@@ -25,5 +25,5 @@
     </joint>
     <!-- base_link -->
-    <!-- <link name="base_footprint">
+    <link name="base_footprint">
         <visual>
             <xacro:insert_mesh_base_link />
@@ -35,7 +35,7 @@
             <xacro:insert_inertia_base_link />
         </inertial>
-    </link> -->
+    </link>
     <!-- imu joint -->
-    <!-- <joint name="imu_fixed" type="fixed">
+    <joint name="imu_fixed" type="fixed">
         <origin xyz="0.0 0 0.45" rpy="0 0 0"/>
         <parent link="base_footprint"/>
@@ -44,5 +44,5 @@
     <link name="imu_link"></link> -->
     <!-- leg link -->
-    <!-- <xacro:human_right_leg parent="base_footprint" dxl_effort="1000" dxl_speed="3"/>
+    <xacro:human_right_leg parent="base_footprint" dxl_effort="1000" dxl_speed="3"/>
     <xacro:human_left_leg parent="base_footprint" dxl_effort="1000" dxl_speed="3"/> -->
 </robot>

File: models/human1.urdf (robot description, URDF)
Before this commit: robot human, 5 links, 4 joints
Links:
- added link r_hip_roll_link, mass 0.342; collision mesh filename=package://human/meshes/r_hip_roll.STL scale=1 1 1; visual mesh filename=package://human/meshes/r_hip_roll.STL scale=1 1 1
Joints:
- added joint r_hip_roll_joint: type revolute, parent r_hip_yaw_link, child r_hip_roll_link, origin xyz=0 0 0 rpy=0 0 0, axis 0 0 1, limit lower=${-pi*0.9} upper=${pi*0.9} effort=1000 velocity=3
- joint r_hip_yaw_joint: limit lower=-2.8274333886 upper=2.8274333886 effort=10000 velocity=3 -> lower=${-pi*0.9} upper=${pi*0.9} effort=1000 velocity=3; origin xyz=0.0 -0.09 -0.068 rpy=0 0 -1.570796327 -> xyz=0 0 0  rpy=0 0 0
